File: Power8Board V1/INA240 Current Sensor 0.kicad_sch (KiCad schematic)
At the start: 3 parts, among them U11 INA240A2PWR

Commit message: Laid out components
Parts:
- removed C33: 0.1 uF, 0805 Ceramic Capacitor:CAPC2012X140N, symbol Device:C_Small
- added C29: 0.1 uF, 0805 Ceramic Capacitor:CAPC2012X140N, symbol Device:C_Small
- added FB11: FerriteBead, MPZ2012S102ATD25:BEADC2012X105N, symbol Device:FerriteBead
Connections:
- net +3.3V: now also FB11.1; no longer U11.5 (VS)
- net GND: now also C29.1
- new net +3.3VA/11: C29.2, FB11.2, U11.5 (VS)
