File: Power8Board V1/INA240 Current Sensor 2.kicad_sch (KiCad schematic)
At the start: 3 parts, among them U5 INA240A2PWR

Commit message: Laid out components
Parts:
- added FB5: FerriteBead, MPZ2012S102ATD25:BEADC2012X105N, symbol Device:FerriteBead
Connections:
- net +3.3V: now also FB5.1; no longer C27.2, U5.5 (VS)
- new net +3.3VA/5: C27.2, FB5.2, U5.5 (VS)
Other:
- moved on the sheet: C27
