File: Power8Board V1/INA240 Current Sensor 5.kicad_sch (KiCad schematic)
At the start: 3 parts, among them U8 INA240A2PWR

Commit message: Laid out components
Parts:
- removed C30: 0.1 uF, 0805 Ceramic Capacitor:CAPC2012X140N, symbol Device:C_Small
- added C10: 0.1 uF, 0805 Ceramic Capacitor:CAPC2012X140N, symbol Device:C_Small
- added FB8: FerriteBead, MPZ2012S102ATD25:BEADC2012X105N, symbol Device:FerriteBead
Connections:
- net +3.3V: now also FB8.1; no longer U8.5 (VS)
- net GND: now also C10.1
- new net +3.3VA/8: C10.2, FB8.2, U8.5 (VS)
