File: Power8Board V1/INA240 Current Sensor 6.kicad_sch (KiCad schematic)
At the start: 3 parts, among them U9 INA240A2PWR

Commit message: Laid out components
Parts:
- removed C31: 0.1 uF, 0805 Ceramic Capacitor:CAPC2012X140N, symbol Device:C_Small
- added C26: 0.1 uF, 0805 Ceramic Capacitor:CAPC2012X140N, symbol Device:C_Small
- added FB9: FerriteBead, MPZ2012S102ATD25:BEADC2012X105N, symbol Device:FerriteBead
Connections:
- net +3.3V: now also FB9.1; no longer U9.5 (VS)
- net GND: now also C26.1
- new net +3.3VA/9: C26.2, FB9.2, U9.5 (VS)
